Commit message: linked to gazebo

File: hexapod_description/model/model.urdf (robot description, URDF)
Before this commit: robot robot_name, 32 links, 31 joints
Links:
- link body: mass 0.01 -> 0.2; geometry collision mesh filename=file:///home/percival/hexapod/install/hexapod_description/s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 scale=1.0 1.0 1.0; visual mesh filename=file:///home/percival/hexapod/install/hexapod_description/s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 scale=1.0 1.0 1.0
- link coxa_l1: geometry collision mesh filename=file:///home/percival/hexapod/install/hexapod_description/s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 scale=1.0 1.0 1.0; visual mesh filename=file:///home/percival/hexapod/install/hexapod_description/s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 scale=1.0 1.0 1.0
- link coxa_l2: geometry collision mesh filename=file:///home/percival/hexapod/install/hexapod_description/s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 scale=1.0 1.0 1.0; visual mesh filename=file:///home/percival/hexapod/install/hexapod_description/s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 scale=1.0 1.0 1.0
- link coxa_l3: geometry collision mesh filename=file:///home/percival/hexapod/install/hexapod_description/s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 scale=1.0 1.0 1.0; visual mesh filename=file:///home/percival/hexapod/install/hexapod_description/s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 scale=1.0 1.0 1.0
- link coxa_r1: geometry collision mesh filename=file:///home/percival/hexapod/install/hexapod_description/s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 scale=1.0 1.0 1.0; visual mesh filename=file:///home/percival/hexapod/install/hexapod_description/s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 scale=1.0 1.0 1.0
- link coxa_r2: geometry collision mesh filename=file:///home/percival/hexapod/install/hexapod_description/s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 scale=1.0 1.0 1.0; visual mesh filename=file:///home/percival/hexapod/install/hexapod_description/s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 scale=1.0 1.0 1.0
- link coxa_r3: geometry collision mesh filename=file:///home/percival/hexapod/install/hexapod_description/s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 scale=1.0 1.0 1.0; visual mesh filename=file:///home/percival/hexapod/install/hexapod_description/s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 scale=1.0 1.0 1.0
- link femur_l1: geometry collision mesh filename=file:///home/percival/hexapod/install/hexapod_description/s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; visual mesh filename=file:///home/percival/hexapod/install/hexapod_description/s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
- link femur_l2: geometry collision mesh filename=file:///home/percival/hexapod/install/hexapod_description/s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; visual mesh filename=file:///home/percival/hexapod/install/hexapod_description/s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
- link femur_l3: geometry collision mesh filename=file:///home/percival/hexapod/install/hexapod_description/s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; visual mesh filename=file:///home/percival/hexapod/install/hexapod_description/s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
- link femur_r1: geometry collision mesh filename=file:///home/percival/hexapod/install/hexapod_description/s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; visual mesh filename=file:///home/percival/hexapod/install/hexapod_description/s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
- link femur_r2: geometry collision mesh filename=file:///home/percival/hexapod/install/hexapod_description/s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; visual mesh filename=file:///home/percival/hexapod/install/hexapod_description/s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
- link femur_r3: geometry collision mesh filename=file:///home/percival/hexapod/install/hexapod_description/s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; visual mesh filename=file:///home/percival/hexapod/install/hexapod_description/s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
- link tibia_foot_l1: geometry collision box size=0.001 0.01 0.01
- link tibia_foot_l2: geometry collision box size=0.001 0.01 0.01
- link tibia_foot_l3: geometry collision box size=0.001 0.01 0.01
- link tibia_foot_r1: geometry collision box size=0.001 0.01 0.01
- link tibia_foot_r2: geometry collision box size=0.001 0.01 0.01
- link tibia_foot_r3: geometry collision box size=0.001 0.01 0.01
- link tibia_l1: geometry collision mesh filename=file:///home/percival/hexapod/install/hexapod_description/s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 scale=1.0 1.0 1.0; visual mesh filename=file:///home/percival/hexapod/install/hexapod_description/s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 scale=1.0 1.0 1.0
- link tibia_l2: geometry collision mesh filename=file:///home/percival/hexapod/install/hexapod_description/s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 scale=1.0 1.0 1.0; visual mesh filename=file:///home/percival/hexapod/install/hexapod_description/s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 scale=1.0 1.0 1.0
- link tibia_l3: geometry collision mesh filename=file:///home/percival/hexapod/install/hexapod_description/s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 scale=1.0 1.0 1.0; visual mesh filename=file:///home/percival/hexapod/install/hexapod_description/s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 scale=1.0 1.0 1.0
- link tibia_r1: geometry collision mesh filename=file:///home/percival/hexapod/install/hexapod_description/s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 scale=1.0 1.0 1.0; visual mesh filename=file:///home/percival/hexapod/install/hexapod_description/s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 scale=1.0 1.0 1.0
- link tibia_r2: geometry collision mesh filename=file:///home/percival/hexapod/install/hexapod_description/s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 scale=1.0 1.0 1.0; visual mesh filename=file:///home/percival/hexapod/install/hexapod_description/s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 scale=1.0 1.0 1.0
- link tibia_r3: geometry collision mesh filename=file:///home/percival/hexapod/install/hexapod_description/s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 scale=1.0 1.0 1.0; visual mesh filename=file:///home/percival/hexapod/install/hexapod_description/s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 scale=1.0 1.0 1.0
Joints:
- joint femur_joint_l1: origin xyz=0.0294 0 0 rpy=-1.57 0 0 -> xyz=0.0294 0 0 rpy=-1.57 0 -0.284
- joint femur_joint_l2: origin xyz=0.0294 0 0 rpy=-1.57 0 0 -> xyz=0.0294 0 0 rpy=-1.57 0 -0.284
- joint femur_joint_l3: origin xyz=0.0294 0 0 rpy=-1.57 0 0 -> xyz=0.0294 0 0 rpy=-1.57 0 -0.284
- joint femur_joint_r1: origin xyz=0.0294 0 0 rpy=-1.57 0 0 -> xyz=0.0294 0 0 rpy=-1.57 0 -0.284
- joint femur_joint_r2: origin xyz=0.0294 0 0 rpy=-1.57 0 0 -> xyz=0.0294 0 0 rpy=-1.57 0 -0.284
- joint femur_joint_r3: origin xyz=0.0294 0 0 rpy=-1.57 0 0 -> xyz=0.0294 0 0 rpy=-1.57 0 -0.284
- joint tibia_foot_joint_l1: origin xyz=0.117 0 0 rpy=0 0 0 -> xyz=0.115 0 0 rpy=0 0 0
- joint tibia_foot_joint_l2: origin xyz=0.117 0 0 rpy=0 0 0 -> xyz=0.115 0 0 rpy=0 0 0
- joint tibia_foot_joint_l3: origin xyz=0.117 0 0 rpy=0 0 0 -> xyz=0.115 0 0 rpy=0 0 0
- joint tibia_foot_joint_r1: origin xyz=0.117 0 0 rpy=0 0 0 -> xyz=0.115 0 0 rpy=0 0 0
- joint tibia_foot_joint_r2: origin xyz=0.117 0 0 rpy=0 0 0 -> xyz=0.115 0 0 rpy=0 0 0
- joint tibia_foot_joint_r3: origin xyz=0.117 0 0 rpy=0 0 0 -> xyz=0.115 0 0 rpy=0 0 0
- joint tibia_joint_l1: origin xyz=0.08 0.0 0.0 rpy=0.0 0.0 0.0 -> xyz=0.08 0.0 0.0 rpy=0.0 0.0 -1.1
- joint tibia_joint_l2: origin xyz=0.08 0.0 0.0 rpy=0.0 0.0 0.0 -> xyz=0.08 0.0 0.0 rpy=0.0 0.0 -1.1
- joint tibia_joint_l3: origin xyz=0.08 0.0 0.0 rpy=0.0 0.0 0.0 -> xyz=0.08 0.0 0.0 rpy=0.0 0.0 -1.1
- joint tibia_joint_r1: origin xyz=0.08 0.0 0.0 rpy=0.0 0.0 0.0 -> xyz=0.08 0.0 0.0 rpy=0.0 0.0 -1.1
- joint tibia_joint_r2: origin xyz=0.08 0.0 0.0 rpy=0.0 0.0 0.0 -> xyz=0.08 0.0 0.0 rpy=0.0 0.0 -1.1
- joint tibia_joint_r3: origin xyz=0.08 0.0 0.0 rpy=0.0 0.0 0.0 -> xyz=0.08 0.0 0.0 rpy=0.0 0.0 -1.1
