Commit message: added controller for each joint

File: hexapod_description/urdf/gazebo.xacro (robot description, xacro)
@@ -4,3 +4,32 @@
         <plugin filename="gz-sim-joint-state-publisher-system" name="gz::sim::systems::JointStatePublisher"/>
     </gazebo>
+    <xacro:macro name="joint_position_controller" params="joint_name initial_position">
+        <gazebo>
+            <plugin filename="gz-sim-joint-position-controller-system" name="gz::sim::systems::JointPositionController">
+                <joint_name>${joint_name}</joint_name>
+                <initial_position>${initial_position}</initial_position>
+                <p_gain>100.0</p_gain>
+                <d_gain>0.0</d_gain>
+                <i_gain>0.0</i_gain>
+            </plugin>
+        </gazebo>
+    </xacro:macro>
+    <xacro:joint_position_controller joint_name="coxa_joint_l1" initial_position="0.0"/>
+    <xacro:joint_position_controller joint_name="coxa_joint_l2" initial_position="0.0"/>
+    <xacro:joint_position_controller joint_name="coxa_joint_l3" initial_position="0.0"/>
+    <xacro:joint_position_controller joint_name="coxa_joint_r1" initial_position="0.0"/>
+    <xacro:joint_position_controller joint_name="coxa_joint_r2" initial_position="0.0"/>
+    <xacro:joint_position_controller joint_name="coxa_joint_r3" initial_position="0.0"/>
+    <xacro:joint_position_controller joint_name="femur_joint_l1" initial_position="0.0"/>
+    <xacro:joint_position_controller joint_name="femur_joint_l2" initial_position="0.0"/>
+    <xacro:joint_position_controller joint_name="femur_joint_l3" initial_position="0.0"/>
+    <xacro:joint_position_controller joint_name="femur_joint_r1" initial_position="0.0"/>
+    <xacro:joint_position_controller joint_name="femur_joint_r2" initial_position="0.0"/>
+    <xacro:joint_position_controller joint_name="femur_joint_r3" initial_position="0.0"/>
+    <xacro:joint_position_controller joint_name="tibia_joint_l1" initial_position="0.0"/>
+    <xacro:joint_position_controller joint_name="tibia_joint_l2" initial_position="0.0"/>
+    <xacro:joint_position_controller joint_name="tibia_joint_l3" initial_position="0.0"/>
+    <xacro:joint_position_controller joint_name="tibia_joint_r1" initial_position="0.0"/>
+    <xacro:joint_position_controller joint_name="tibia_joint_r2" initial_position="0.0"/>
+    <xacro:joint_position_controller joint_name="tibia_joint_r3" initial_position="0.0"/>
 </robot>

File: hexapod_description/urdf/links.xacro (robot description, xacro)
@@ -1,4 +1,7 @@
 <?xml version="1.0"?>
 <robot xmlns:xacro="http://www.ros.org/wiki/xacro">
+    <xacro:property name="friction" value="0.4"/>
+    <xacro:property name="joint_vel" value="2.0"/>
+    <xacro:property name="joint_effort" value="100.0"/>
     <link name="base_link"/>
     <joint name="base_joint" type="fixed">
@@ -34,5 +37,6 @@
             <child link="coxa_${side}${num}"/>
             <axis xyz="0 0 -1"/>
-            <limit lower="-1.5" upper="1.5" velocity="100.0" effort="1000.0"/>
+            <limit lower="-1.04" upper="1.04" velocity="${joint_vel}" effort="${joint_effort}"/>
+            <dynamics damping="0.0" friction="${friction}"/>
             <origin xyz="0 0 0" rpy="0 0 ${ang}"/>
         </joint>
@@ -57,5 +61,6 @@
             <child link="femur_${side}${num}"/>
             <axis xyz="0 0 -1"/>
-            <limit lower="-1.5" upper="1.5" velocity="100.0" effort="1000.0"/>
+            <limit lower="-1.04" upper="1.04" velocity="${joint_vel}" effort="${joint_effort}"/>
+            <dynamics damping="0.0" friction="${friction}"/>
             <origin xyz="0.0882 0 0" rpy="-1.57 0 0"/>
         </joint>
@@ -81,5 +86,6 @@
             <child link="tibia_${side}${num}"/>
             <axis xyz="0 0 1"/>
-            <limit lower="-1.5" upper="1.5" velocity="100.0" effort="1000.0"/>
+            <limit lower="-0.7" upper="1.57" velocity="${joint_vel}" effort="${joint_effort}"/>
+            <dynamics damping="0.0" friction="${friction}"/>
         </joint>
         <link name="tibia_${side}${num}">
@@ -105,18 +111,4 @@
             <xacro:box_inertia m="0.015" x="0.3" y="0.05" z="0.05" o_xyz="-0.035 0.0 ${tibia_box_z_val}" o_rpy="0 0 0"/>
         </link>
-        <joint name="tibia_foot_joint_${side}${num}" type="fixed">
-    		<origin xyz="0.345 0 0" rpy="0 0 0" />
-    		<parent link="tibia_${side}${num}" />
-    		<child link="tibia_foot_${side}${num}" />
-  	    </joint>
-        <link name="tibia_foot_${side}${num}">
-            <collision>
-                <origin xyz="0.0 0.0 0.0" rpy="0.0 0.0 0.0"/>
-                <geometry>
-                    <box size="0.001 0.01 0.01"/>
-                </geometry>
-            </collision>
-		    <xacro:box_inertia m="0.001" x="0.001" y="0.01" z="0.01" o_xyz="0 0 0" o_rpy="0 0 0"/>
-  	    </link>
     </xacro:macro>
     <xacro:leg side="r" num="1" coxa_y_val = "-0.03" femur_z_val = "0.067" tibia_box_z_val = "0.008" x="0.262794" 	y="-0.151725" 	ang="-${pi/3}" />
